File: Hardware/MMS hat dummy.kicad_pcb (KiCad board)
At the start: 2 copper layers, 100 x 20 mm, 26 parts, among them J1 Chainbus in, J2 Chainbus Out, U1 XC6206P332MR

Commit message: added documentation
Other:
- board text added: "MMS3 Hat Dummy (Led's optional) V1.0, Made By Wojciech Szafrański"
- board text removed: "MMS3 Hat Dummy (Led's optional) Made By Wojciech Szafrański"
Changed lines of the file:
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@@
 		(layer "Edge.Cuts")
 	)
-	(gr_text "MMS3 Hat Dummy\n(Led's optional)\nMade By\nWojciech Szafrański"
+	(gr_text "MMS3 Hat Dummy\n(Led's optional)\nV1.0, Made By\nWojciech Szafrański"
 		(at 176 106 0)
 		(layer "F.SilkS")

Commit message: fixed reserved pins
Connections:
- J1 pad 25: unconnected-(J1-Pin_25-Pad25) -> /R1
- J1 pad 27: unconnected-(J1-Pin_27-Pad27) -> /R2
- J2 pad 25: unconnected-(J2-Pin_25-Pad25) -> /R1
- J2 pad 27: unconnected-(J2-Pin_27-Pad27) -> /R2
Routing:
- net /R1: track 0.00 -> 2.81 mm, vias 0 -> 1
- net /R2: track 0.00 -> 2.59 mm, vias 0 -> 1
Other:
- board text added: "MMS3 Hat Dummy (Led's optional) V1.1, Made By Wojciech Szafrański"
- board text removed: "MMS3 Hat Dummy (Led's optional) V1.0, Made By Wojciech Szafrański"
Changed lines of the file:
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@@
 			(size 3 1)
 			(layers "F.Cu" "F.Mask" "F.Paste")
-			(net "unconnected-(J2-Pin_25-Pad25)")
+			(net "/R1")
 			(pinfunction "Pin_25_25")
-			(pintype "passive+no_connect")
+			(pintype "passive")
 		)
 		(pad "26" smd rect
@@
 			(size 3 1)
 			(layers "F.Cu" "F.Mask" "F.Paste")
-			(net "unconnected-(J2-Pin_27-Pad27)")
+			(net "/R2")
 			(pinfunction "Pin_27_27")
-			(pintype "passive+no_connect")
+			(pintype "passive")
 		)
 		(pad "28" smd rect
@@
 			(size 3.15 1)
 			(layers "B.Cu" "B.Mask" "B.Paste")
-			(net "unconnected-(J1-Pin_25-Pad25)")
+			(net "/R1")
 			(pinfunction "Pin_25_25")
-			(pintype "passive+no_connect")
+			(pintype "passive")
 		)
 		(pad "26" smd rect
@@
 			(size 3.15 1)
 			(layers "B.Cu" "B.Mask" "B.Paste")
-			(net "unconnected-(J1-Pin_27-Pad27)")
+			(net "/R2")
 			(pinfunction "Pin_27_27")
-			(pintype "passive+no_connect")
+			(pintype "passive")
 		)
 		(pad "28" smd rect
@@
 		(layer "Edge.Cuts")
 	)
-	(gr_text "MMS3 Hat Dummy\n(Led's optional)\nV1.0, Made By\nWojciech Szafrański"
+	(gr_text "MMS3 Hat Dummy\n(Led's optional)\nV1.1, Made By\nWojciech Szafrański"
 		(at 176 106 0)
 		(layer "F.SilkS")
@@
 		(net "/Chainbus.RX")
 	)
+	(segment
+		(start 138.961728 93.038272)
+		(end 138.3 93.7)
+		(width 0.2)
+		(layer "F.Cu")
+		(net "/R1")
+	)
+	(segment
+		(start 139.43 93.038272)
+		(end 138.961728 93.038272)
+		(width 0.2)
+		(layer "F.Cu")
+		(net "/R1")
+	)
+	(via
+		(at 138.3 93.7)
+		(size 0.5)
+		(drill 0.3)
+		(layers "F.Cu" "B.Cu")
+		(net "/R1")
+	)
+	(segment
+		(start 138.733272 93.7)
+		(end 139.42 93.013272)
+		(width 0.2)
+		(layer "B.Cu")
+		(net "/R1")
+	)
+	(segment
+		(start 138.3 93.7)
+		(end 138.733272 93.7)
+		(width 0.2)
+		(layer "B.Cu")
+		(net "/R1")
+	)
+	(segment
+		(start 141.97 93.038272)
+		(end 141.611728 93.038272)
+		(width 0.2)
+		(layer "F.Cu")
+		(net "/R2")
+	)
+	(segment
+		(start 141.611728 93.038272)
+		(end 140.95 93.7)
+		(width 0.2)
+		(layer "F.Cu")
+		(net "/R2")
+	)
+	(via
+		(at 140.95 93.7)
+		(size 0.5)
+		(drill 0.3)
+		(layers "F.Cu" "B.Cu")
+		(net "/R2")
+	)
+	(segment
+		(start 141.273272 93.7)
+		(end 141.96 93.013272)
+		(width 0.2)
+		(layer "B.Cu")
+		(net "/R2")
+	)
+	(segment
+		(start 140.95 93.7)
+		(end 141.273272 93.7)
+		(width 0.2)
+		(layer "B.Cu")
+		(net "/R2")
+	)
 	(zone
