File: Hardware/MMS hat dummy.kicad_sch (KiCad schematic)
At the start: 25 parts, among them J1 Chainbus in, J2 Chainbus Out, U1 XC6206P332MR

Commit message: fixed reserved pins
Connections:
- net R1: now reaches J2.25 (Pin_25)
- net R1: now also J1.25 (Pin_25)
- net R2: now reaches J2.27 (Pin_27)
- net R2: now also J1.27 (Pin_27)
- no-connect marks 4 -> 0
Changed lines of the file:
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@@
 		(color 0 0 0 0)
 	)
-	(no_connect
-		(at 149.86 74.93)
-	)
-	(no_connect
-		(at 71.12 74.93)
-	)
-	(no_connect
-		(at 147.32 74.93)
-	)
-	(no_connect
-		(at 73.66 74.93)
-	)
 	(bus_entry
 		(at 142.24 106.68)
@@
 			(width 0)
 			(type default)
+		)
+	)
+	(label "R2"
+		(at 73.66 74.93 0)
+		(effects
+			(font
+				(size 1.27 1.27)
+			)
+			(justify left bottom)
 		)
 	)
@@
 		)
 	)
+	(label "R2"
+		(at 149.86 74.93 0)
+		(effects
+			(font
+				(size 1.27 1.27)
+			)
+			(justify left bottom)
+		)
+	)
 	(label "SEL1"
 		(at 40.64 97.79 270)
@@
 		)
 	)
+	(label "R1"
+		(at 71.12 74.93 0)
+		(effects
+			(font
+				(size 1.27 1.27)
+			)
+			(justify left bottom)
+		)
+	)
 	(label "SEL8"
 		(at 58.42 97.79 270)
@@
 		)
 	)
+	(label "R1"
+		(at 147.32 74.93 0)
+		(effects
+			(font
+				(size 1.27 1.27)
+			)
+			(justify left bottom)
+		)
+	)
